File: Interface HW-01.sch (KiCad schematic (older format))
At the start: 35 parts

Commit message: Working on adding new page, intermediate commit
Connections:
- net labels added: +15V, -15V, DAC_X+, DAC_X-, DAC_Y+, DAC_Y-
- net labels removed: DAC_X
- wire segments 138 -> 154
Changed lines of the file:
@@
 Sheet 1 1
 Title "Defcon Bot Interface Brd"
-Date "27 mar 2014"
+Date "1 apr 2014"
 Rev "1"
 Comp ""
@@
 	1    0    0    -1
 $EndComp
-Wire Wire Line
-	2100 3800 2550 3800
 $Comp
 L 74XXX1G32 U?
@@
 $EndComp
 Wire Wire Line
-	2050 5950 2500 5950
-Wire Wire Line
 	750  3750 1400 3750
 Text Label 850  3750 0    60   ~ 0
@@
 U 1 1 5332472C
 P 5550 3350
-F 0 "R?" H 5650 3300 50  0000 C CNN
-F 1 "R_US" H 5700 3400 50  0000 C CNN
+F 0 "R?" H 5650 3400 50  0000 C CNN
+F 1 "R_US" H 5700 3300 50  0000 C CNN
 F 2 "" H 5550 3350 60  0000 C CNN
 F 3 "" H 5550 3350 60  0000 C CNN
@@
 	4550 6900 4850 6900
 Connection ~ 4550 6150
-Text GLabel 8200 2400 0    60   Input ~ 0
-DAC_X
+Text GLabel 7550 2350 2    60   Input ~ 0
+DAC_X+
+Wire Wire Line
+	2050 3800 2550 3800
+Wire Wire Line
+	2000 5950 2500 5950
+$Comp
+L +15V #PWR?
+U 1 1 533B46C7
+P 6250 1900
+F 0 "#PWR?" H 6250 1850 20  0001 C CNN
+F 1 "+15V" H 6250 2000 30  0000 C CNN
+F 2 "~" H 6250 1900 60  0000 C CNN
+F 3 "~" H 6250 1900 60  0000 C CNN
+	1    6250 1900
+	1    0    0    -1
+$EndComp
+Wire Wire Line
+	6250 1950 6250 1900
+$Comp
+L -15V #PWR?
+U 1 1 533B4779
+P 6400 2750
+F 0 "#PWR?" H 6400 2700 20  0001 C CNN
+F 1 "-15V" H 6400 2850 30  0000 C CNN
+F 2 "~" H 6400 2750 60  0000 C CNN
+F 3 "~" H 6400 2750 60  0000 C CNN
+	1    6400 2750
+	1    0    0    -1
+$EndComp
+Wire Wire Line
+	6250 2750 6250 2800
+Wire Wire Line
+	6250 2800 6400 2800
+Wire Wire Line
+	6400 2800 6400 2750
+$Comp
+L +15V #PWR?
+U 1 1 533B48D2
+P 6250 3350
+F 0 "#PWR?" H 6250 3300 20  0001 C CNN
+F 1 "+15V" H 6250 3450 30  0000 C CNN
+F 2 "~" H 6250 3350 60  0000 C CNN
+F 3 "~" H 6250 3350 60  0000 C CNN
+	1    6250 3350
+	1    0    0    -1
+$EndComp
+Wire Wire Line
+	6250 3400 6250 3350
+$Comp
+L +15V #PWR?
+U 1 1 533B48D9
+P 6250 4800
+F 0 "#PWR?" H 6250 4750 20  0001 C CNN
+F 1 "+15V" H 6250 4900 30  0000 C CNN
+F 2 "~" H 6250 4800 60  0000 C CNN
+F 3 "~" H 6250 4800 60  0000 C CNN
+	1    6250 4800
+	1    0    0    -1
+$EndComp
+Wire Wire Line
+	6250 4850 6250 4800
+$Comp
+L +15V #PWR?
+U 1 1 533B48E0
+P 6250 6250
+F 0 "#PWR?" H 6250 6200 20  0001 C CNN
+F 1 "+15V" H 6250 6350 30  0000 C CNN
+F 2 "~" H 6250 6250 60  0000 C CNN
+F 3 "~" H 6250 6250 60  0000 C CNN
+	1    6250 6250
+	1    0    0    -1
+$EndComp
+Wire Wire Line
+	6250 6300 6250 6250
+$Comp
+L -15V #PWR?
+U 1 1 533B48E7
+P 6400 4200
+F 0 "#PWR?" H 6400 4150 20  0001 C CNN
+F 1 "-15V" H 6400 4300 30  0000 C CNN
+F 2 "~" H 6400 4200 60  0000 C CNN
+F 3 "~" H 6400 4200 60  0000 C CNN
+	1    6400 4200
+	1    0    0    -1
+$EndComp
+$Comp
+L -15V #PWR?
+U 1 1 533B48ED
+P 6400 5650
+F 0 "#PWR?" H 6400 5600 20  0001 C CNN
+F 1 "-15V" H 6400 5750 30  0000 C CNN
+F 2 "~" H 6400 5650 60  0000 C CNN
+F 3 "~" H 6400 5650 60  0000 C CNN
+	1    6400 5650
+	1    0    0    -1
+$EndComp
+$Comp
+L -15V #PWR?
+U 1 1 533B48F3
+P 6400 7100
+F 0 "#PWR?" H 6400 7050 20  0001 C CNN
+F 1 "-15V" H 6400 7200 30  0000 C CNN
+F 2 "~" H 6400 7100 60  0000 C CNN
+F 3 "~" H 6400 7100 60  0000 C CNN
+	1    6400 7100
+	1    0    0    -1
+$EndComp
+Wire Wire Line
+	6250 7100 6250 7150
+Wire Wire Line
+	6250 7150 6400 7150
+Wire Wire Line
+	6400 7150 6400 7100
+Wire Wire Line
+	6250 5700 6400 5700
+Wire Wire Line
+	6400 5700 6400 5650
+Wire Wire Line
+	6250 5700 6250 5650
+Wire Wire Line
+	6250 4200 6250 4250
+Wire Wire Line
+	6250 4250 6400 4250
+Wire Wire Line
+	6400 4250 6400 4200
+Text GLabel 7550 3800 2    60   Input ~ 0
+DAC_X-
+Text GLabel 7550 5250 2    60   Input ~ 0
+DAC_Y+
+Text GLabel 7550 6700 2    60   Input ~ 0
+DAC_Y-
 $EndSCHEMATC

Commit message: Still working
Parts:
- removed C? (x2): 0.1uF, ~, symbol CSMALL
- removed J? (x3): CONN_8, ~, symbol CONN_8
- removed R? (x17): R_US, symbol R_US
- removed U?: DACX311, symbol DACX311
- removed U? (x4): OPA237, symbol OPA237
- removed U?: 74XXX1G32, symbol 74XXX1G32
- added C? (x6): 0.1uF, ~, symbol CSMALL
- added J? (x3): CONN_8, ~, symbol CONN_8
- added J?: CONN_13X2, ~, symbol CONN_13X2
- added J?: TE: 640456-3, ~, symbol CONN_3
- added R?: 2.2k, symbol R_US
- added TP? (x2): TEST, symbol CONNECTOR
- added U?: DACX311, symbol DACX311
- added U?: 74XXX1G32, symbol 74XXX1G32
- C?: Voltage (none) -> 50V
- R?: value R_US -> 2.2k; Tolerance (none) -> 1%
Connections:
- net labels added: DAC_X, DAC_Y, REF_1.65V
- net labels removed: DAC_X+, DAC_X-, DAC_Y+, DAC_Y-
- wire segments 154 -> 116
Other:
- note added: "POWER INPUT FROM \nGALVO POWER SUPPLY\n"
- note added: "RASPBERRY PI HAS TWO SLAVE SELECT PINS, OR GATES ARE \nNOT NEEDED. SCL_A/SDA_A ARE SLAVE SELECT, SPISTE_A \nIS GPIO"
- moved on the sheet: R?, TP?, U?

Commit message: Modified schematic, added laser driver and page for buck converter
Parts:
- added P?: CONNECTOR_2, symbol CONNECTOR_2
- added Q?: 2N7002, ~, symbol MOS_N
- added R?: 0.0, symbol R_US
- added R?: 2.2k, symbol R_US
Connections:
- wire segments 116 -> 142
Other:
- note added: "LASER MODULE HAS INTERNAL \n700 OHM RESTISTOR, 0 OHM \nADDED IN CASE DIFFERENT \nLASER IS USED"
Changed lines of the file:
@@
 $Descr A 11000 8500
 encoding utf-8
-Sheet 2 4
+Sheet 2 5
 Title "Defcon Bot Interface Brd"
-Date "2 apr 2014"
+Date "5 apr 2014"
 Rev "1"
 Comp ""
@@
 $EndComp
 Wire Wire Line
-	5850 1350 5850 1550
+	5850 1350 5850 1450
+Wire Wire Line
+	5850 1450 5850 1550
 Connection ~ 5850 1450
 Wire Wire Line
@@
 $EndComp
 Wire Wire Line
-	2650 6500 2650 6700
+	2650 6500 2650 6600
+Wire Wire Line
+	2650 6600 2650 6700
 Wire Wire Line
 	3100 6600 2650 6600
@@
 $EndComp
 Wire Wire Line
-	4950 2400 4950 2700
+	4950 2400 4950 2450
+Wire Wire Line
+	4950 2450 4950 2700
 Wire Wire Line
 	4950 2700 4900 2700
@@
 $EndComp
 Wire Wire Line
-	4900 4250 4900 4550
+	4900 4250 4900 4300
+Wire Wire Line
+	4900 4300 4900 4550
 Wire Wire Line
 	4900 4550 4850 4550
@@
 	3650 6300 3650 6400
 Wire Wire Line
-	3500 6000 3500 6300
+	3500 6000 3500 6050
+Wire Wire Line
+	3500 6050 3500 6300
 Connection ~ 3500 6050
 $Comp
@@
 	3100 4550 3600 4550
 Wire Wire Line
-	4100 6700 4650 6700
+	4100 6700 4250 6700
+Wire Wire Line
+	4250 6700 4350 6700
+Wire Wire Line
+	4350 6700 4650 6700
 Text GLabel 4650 6700 2    60   Input ~ 0
 REF_1.65V
@@
 DAC_X
 Wire Wire Line
-	4900 2900 5600 2900
+	4900 2900 5350 2900
+Wire Wire Line
+	5350 2900 5600 2900
 $Comp
 L CONNECTOR TP?
@@
 DAC_Y
 Wire Wire Line
-	4850 4750 5550 4750
+	4850 4750 5300 4750
+Wire Wire Line
+	5300 4750 5550 4750
 $Comp
 L CONNECTOR TP?
@@
 	8200 1200 8100 1200
 Wire Wire Line
-	8100 1200 8100 2150
+	8100 1200 8100 2000
+Wire Wire Line
+	8100 2000 8100 2150
 Wire Wire Line
 	8200 2000 8100 2000
@@
 	9000 1000 9100 1000
 Wire Wire Line
-	9100 1000 9100 2150
+	9100 1000 9100 1400
+Wire Wire Line
+	9100 1400 9100 1700
+Wire Wire Line
+	9100 1700 9100 2150
 Wire Wire Line
 	9000 1400 9100 1400
@@
 	8000 1600 8200 1600
 Wire Wire Line
-	8000 750  8000 1600
+	8000 750  8000 800
+Wire Wire Line
+	8000 800  8000 1600
 Wire Wire Line
 	8200 800  8000 800
@@
 	7150 3850 7300 3850
 Wire Wire Line
-	7300 3800 7300 3900
+	7300 3800 7300 3850
+Wire Wire Line
+	7300 3850 7300 3900
 Connection ~ 7300 3850
 $Comp
@@
 $EndComp
 Wire Wire Line
-	2600 1950 2600 2350
+	2600 1950 2600 2000
+Wire Wire Line
+	2600 2000 2600 2350
 Wire Wire Line
 	2750 2050 2750 2000
@@
 $EndComp
 Wire Wire Line
-	2600 3800 2600 4200
+	2600 3800 2600 3850
+Wire Wire Line
+	2600 3850 2600 4200
 Wire Wire Line
 	2750 3850 2600 3850
@@
 Wire Wire Line
 	2600 3050 2600 3100
+$Comp
+L MOS_N Q?
+U 1 1 53403CA2
+P 8750 5850
+F 0 "Q?" H 8550 6050 30  0000 L CNN
+F 1 "2N7002" H 8550 6000 30  0000 L CNN
+F 2 "~" H 8750 5850 60  0000 C CNN
+F 3 "~" H 8750 5850 60  0000 C CNN
+	1    8750 5850
+	1    0    0    -1
+$EndComp
+$Comp
+L GND #PWR?
+U 1 1 53403CAF
+P 8850 6350
+F 0 "#PWR?" H 8850 6350 30  0001 C CNN
+F 1 "GND" H 8850 6280 30  0001 C CNN
+F 2 "" H 8850 6350 60  0000 C CNN
+F 3 "" H 8850 6350 60  0000 C CNN
+	1    8850 6350
+	1    0    0    -1
+$EndComp
+Wire Wire Line
+	8850 6350 8850 6050
+$Comp
+L CONNECTOR_2 P?
+U 1 1 53403D3C
+P 9200 5050
+F 0 "P?" H 9200 5200 50  0000 L CNN
+F 1 "CONNECTOR_2" H 9200 4900 50  0000 L CNN
+F 2 "" H 9200 5050 60  0000 C CNN
+F 3 "" H 9200 5050 60  0000 C CNN
+	1    9200 5050
+	1    0    0    -1
+$EndComp
+$Comp
+L R_US R?
+U 1 1 53403D4A
+P 8850 5350
+F 0 "R?" H 8900 5400 30  0000 L CNN
+F 1 "0.0" H 8900 5350 30  0000 L CNN
+F 2 "" H 8850 5350 60  0000 C CNN
+F 3 "" H 8850 5350 60  0000 C CNN
+F 4 "5%" H 8900 5300 30  0000 L CNN "Tolerance"
+	1    8850 5350
+	1    0    0    -1
+$EndComp
+Wire Wire Line
+	9150 5100 8850 5100
+Wire Wire Line
+	8850 5100 8850 5150
+Wire Wire Line
+	8850 5650 8850 5550
+$Comp
+L 3V3 #PWR?
+U 1 1 53403E6A
+P 8850 4850
+F 0 "#PWR?" H 8850 4950 40  0001 C CNN
+F 1 "3V3" H 8850 4975 40  0000 C CNN
+F 2 "" H 8850 4850 60  0000 C CNN
+F 3 "" H 8850 4850 60  0000 C CNN
+	1    8850 4850
+	1    0    0    -1
+$EndComp
+Wire Wire Line
+	9150 5000 8850 5000
+Wire Wire Line
+	8850 5000 8850 4850
+Text Notes 9050 5650 0    60   ~ 0
+LASER MODULE HAS INTERNAL \n700 OHM RESTISTOR, 0 OHM \nADDED IN CASE DIFFERENT \nLASER IS USED
+Wire Wire Line
+	7900 5850 8050 5850
+Wire Wire Line
+	8050 5850 8550 5850
+Text Label 8050 5850 0    60   ~ 0
+GPIO_12
+$Comp
+L R_US R?
+U 1 1 53403EFD
+P 8050 6100
+F 0 "R?" H 8100 6150 30  0000 L CNN
+F 1 "2.2k" H 8100 6100 30  0000 L CNN
+F 2 "" H 8050 6100 60  0000 C CNN
+F 3 "" H 8050 6100 60  0000 C CNN
+F 4 "1%" H 8100 6050 30  0000 L CNN "Tolerance"
+	1    8050 6100
+	1    0    0    -1
+$EndComp
+Wire Wire Line
+	8050 5900 8050 5850
+Connection ~ 8050 5850
+$Comp
+L GND #PWR?
+U 1 1 53403F8F
+P 8050 6350
+F 0 "#PWR?" H 8050 6350 30  0001 C CNN
+F 1 "GND" H 8050 6280 30  0001 C CNN
+F 2 "" H 8050 6350 60  0000 C CNN
+F 3 "" H 8050 6350 60  0000 C CNN
+	1    8050 6350
+	1    0    0    -1
+$EndComp
+Wire Wire Line
+	8050 6300 8050 6350
 $EndSCHEMATC

Commit message: Started layout
Parts:
- gave numbers to parts that had none: 27
Connections:
- wire segments 142 -> 126
- no-connect marks 0 -> 13

Commit message: Added a cap to ref, chages buck converter caps, more routing, didn't pull in netlist
Parts:
- added C31: 0.1uF, ~, symbol CSMALL
Connections:
- wire segments 126 -> 128
Changed lines of the file:
@@
 Sheet 2 5
 Title "Connector, DAC, Power Input"
-Date "9 apr 2014"
+Date "16 apr 2014"
 Rev "1"
 Comp ""
@@
 	2650 6500 2650 6700
 Wire Wire Line
-	3100 6600 2650 6600
+	2350 6600 3100 6600
 Connection ~ 2650 6600
 $Comp
@@
 Wire Wire Line
 	9000 1600 9600 1600
+$Comp
+L CSMALL C31
+U 1 1 534DFA1A
+P 2350 6900
+F 0 "C31" H 2450 6950 30  0000 L CNN
+F 1 "0.1uF" H 2450 6900 30  0000 L CNN
+F 2 "~" H 2350 6900 60  0000 C CNN
+F 3 "~" H 2350 6900 60  0000 C CNN
+F 4 "50V" H 2450 6850 30  0000 L CNN "Voltage"
+	1    2350 6900
+	1    0    0    -1
+$EndComp
+Wire Wire Line
+	2350 6800 2350 6600
+$Comp
+L GND #PWR032
+U 1 1 534DFB65
+P 2350 7200
+F 0 "#PWR032" H 2350 7200 30  0001 C CNN
+F 1 "GND" H 2350 7130 30  0001 C CNN
+F 2 "" H 2350 7200 60  0000 C CNN
+F 3 "" H 2350 7200 60  0000 C CNN
+	1    2350 7200
+	1    0    0    -1
+$EndComp
+Wire Wire Line
+	2350 7000 2350 7200
 $EndSCHEMATC

Commit message: More routing, added power supply test points, added mounting holes
Parts:
- added TP4, TP5, TP6, TP7, TP8: TEST, symbol CONNECTOR
Connections:
- wire segments 128 -> 135
Changed lines of the file:
@@
 L CSMALL C6
 U 1 1 533B6223
-P 7300 3700
-F 0 "C6" H 7400 3750 30  0000 L CNN
-F 1 "0.1uF" H 7400 3700 30  0000 L CNN
-F 2 "~" H 7300 3700 60  0000 C CNN
-F 3 "~" H 7300 3700 60  0000 C CNN
-F 4 "50V" H 7400 3650 30  0000 L CNN "Voltage"
-	1    7300 3700
+P 7050 3700
+F 0 "C6" H 7150 3750 30  0000 L CNN
+F 1 "0.1uF" H 7150 3700 30  0000 L CNN
+F 2 "~" H 7050 3700 60  0000 C CNN
+F 3 "~" H 7050 3700 60  0000 C CNN
+F 4 "50V" H 7150 3650 30  0000 L CNN "Voltage"
+	1    7050 3700
 	1    0    0    -1
 $EndComp
@@
 L CSMALL C7
 U 1 1 533B622A
-P 7300 4000
-F 0 "C7" H 7400 4050 30  0000 L CNN
-F 1 "0.1uF" H 7400 4000 30  0000 L CNN
-F 2 "~" H 7300 4000 60  0000 C CNN
-F 3 "~" H 7300 4000 60  0000 C CNN
-F 4 "50V" H 7400 3950 30  0000 L CNN "Voltage"
-	1    7300 4000
+P 7050 4000
+F 0 "C7" H 7150 4050 30  0000 L CNN
+F 1 "0.1uF" H 7150 4000 30  0000 L CNN
+F 2 "~" H 7050 4000 60  0000 C CNN
+F 3 "~" H 7050 4000 60  0000 C CNN
+F 4 "50V" H 7150 3950 30  0000 L CNN "Voltage"
+	1    7050 4000
 	1    0    0    -1
 $EndComp
@@
 L GND #PWR020
 U 1 1 533B6230
-P 7150 3900
-F 0 "#PWR020" H 7150 3900 30  0001 C CNN
-F 1 "GND" H 7150 3830 30  0001 C CNN
-F 2 "" H 7150 3900 60  0000 C CNN
-F 3 "" H 7150 3900 60  0000 C CNN
-	1    7150 3900
-	1    0    0    -1
-$EndComp
-Wire Wire Line
-	7150 3900 7150 3850
-Wire Wire Line
-	7150 3850 7300 3850
-Wire Wire Line
-	7300 3800 7300 3900
-Connection ~ 7300 3850
+P 6900 3900
+F 0 "#PWR020" H 6900 3900 30  0001 C CNN
+F 1 "GND" H 6900 3830 30  0001 C CNN
+F 2 "" H 6900 3900 60  0000 C CNN
+F 3 "" H 6900 3900 60  0000 C CNN
+	1    6900 3900
+	1    0    0    -1
+$EndComp
+Wire Wire Line
+	6900 3900 6900 3850
+Wire Wire Line
+	6900 3850 7050 3850
+Wire Wire Line
+	7050 3800 7050 3900
+Connection ~ 7050 3850
 $Comp
 L +15V #PWR021
 U 1 1 533B6324
-P 7300 3550
-F 0 "#PWR021" H 7300 3500 20  0001 C CNN
-F 1 "+15V" H 7300 3650 30  0000 C CNN
-F 2 "~" H 7300 3550 60  0000 C CNN
-F 3 "~" H 7300 3550 60  0000 C CNN
-	1    7300 3550
-	1    0    0    -1
-$EndComp
-Wire Wire Line
-	7300 3600 7300 3550
+P 7050 3500
+F 0 "#PWR021" H 7050 3450 20  0001 C CNN
+F 1 "+15V" H 7050 3600 30  0000 C CNN
+F 2 "~" H 7050 3500 60  0000 C CNN
+F 3 "~" H 7050 3500 60  0000 C CNN
+	1    7050 3500
+	1    0    0    -1
+$EndComp
+Wire Wire Line
+	7050 3600 7050 3500
 $Comp
 L -15V #PWR022
 U 1 1 533B63A2
-P 7300 4150
-F 0 "#PWR022" H 7300 4100 20  0001 C CNN
-F 1 "-15V" H 7300 4250 30  0000 C CNN
-F 2 "~" H 7300 4150 60  0000 C CNN
-F 3 "~" H 7300 4150 60  0000 C CNN
-	1    7300 4150
+P 7050 4200
+F 0 "#PWR022" H 7050 4150 20  0001 C CNN
+F 1 "-15V" H 7050 4300 30  0000 C CNN
+F 2 "~" H 7050 4200 60  0000 C CNN
+F 3 "~" H 7050 4200 60  0000 C CNN
+	1    7050 4200
 	-1   0    0    1
 $EndComp
 Wire Wire Line
-	7300 4100 7300 4150
+	7050 4100 7050 4200
 Wire Wire Line
 	8200 3950 8050 3950
@@
 Wire Wire Line
 	2350 7000 2350 7200
+$Comp
+L CONNECTOR TP5
+U 1 1 534E035D
+P 6750 6250
+F 0 "TP5" H 6900 6350 30  0000 L CNN
+F 1 "TEST" H 6900 6300 30  0000 L CNN
+F 2 "" H 6750 6250 60  0000 C CNN
+F 3 "" H 6750 6250 60  0000 C CNN
+	1    6750 6250
+	1    0    0    -1
+$EndComp
+$Comp
+L CONNECTOR TP6
+U 1 1 534E0363
+P 6750 6400
+F 0 "TP6" H 6900 6500 30  0000 L CNN
+F 1 "TEST" H 6900 6450 30  0000 L CNN
+F 2 "" H 6750 6400 60  0000 C CNN
+F 3 "" H 6750 6400 60  0000 C CNN
+	1    6750 6400
+	1    0    0    -1
+$EndComp
+$Comp
+L GND #PWR033
+U 1 1 534E0369
+P 6600 6500
+F 0 "#PWR033" H 6600 6500 30  0001 C CNN
+F 1 "GND" H 6600 6430 30  0001 C CNN
+F 2 "" H 6600 6500 60  0000 C CNN
+F 3 "" H 6600 6500 60  0000 C CNN
+	1    6600 6500
+	1    0    0    -1
+$EndComp
+Wire Wire Line
+	6600 6250 6600 6500
+Wire Wire Line
+	6700 6250 6600 6250
+Wire Wire Line
+	6700 6400 6600 6400
+Connection ~ 6600 6400
+$Comp
+L CONNECTOR TP4
+U 1 1 534E0497
+P 6750 5950
+F 0 "TP4" H 6900 6050 30  0000 L CNN
+F 1 "TEST" H 6900 6000 30  0000 L CNN
+F 2 "" H 6750 5950 60  0000 C CNN
+F 3 "" H 6750 5950 60  0000 C CNN
+	1    6750 5950
+	1    0    0    -1
+$EndComp
+$Comp
+L 3V3 #PWR034
+U 1 1 534E049D
+P 6600 5900
+F 0 "#PWR034" H 6600 6000 40  0001 C CNN
+F 1 "3V3" H 6600 6025 40  0000 C CNN
+F 2 "" H 6600 5900 60  0000 C CNN
+F 3 "" H 6600 5900 60  0000 C CNN
+	1    6600 5900
+	1    0    0    -1
+$EndComp
+Wire Wire Line
+	6600 5900 6600 5950
+Wire Wire Line
+	6600 5950 6700 5950
+$Comp
+L CONNECTOR TP7
+U 1 1 534E054C
+P 7200 3550
+F 0 "TP7" H 7350 3650 30  0000 L CNN
+F 1 "TEST" H 7350 3600 30  0000 L CNN
+F 2 "" H 7200 3550 60  0000 C CNN
+F 3 "" H 7200 3550 60  0000 C CNN
+	1    7200 3550
+	1    0    0    -1
+$EndComp
+Wire Wire Line
+	7150 3550 7050 3550
+Connection ~ 7050 3550
+$Comp
+L CONNECTOR TP8
+U 1 1 534E05FD
+P 7200 4150
+F 0 "TP8" H 7350 4250 30  0000 L CNN
+F 1 "TEST" H 7350 4200 30  0000 L CNN
+F 2 "" H 7200 4150 60  0000 C CNN
+F 3 "" H 7200 4150 60  0000 C CNN
+	1    7200 4150
+	1    0    0    -1
+$EndComp
+Wire Wire Line
+	7150 4150 7050 4150
+Connection ~ 7050 4150
 $EndSCHEMATC
