File: Interface HW-01.sch (KiCad schematic (older format))
At the start: 33 parts, among them J1 CONN_8, J2 CONN_8, J3 CONN_8, J4 CONN_8, J5 TE: 640456-3, J6 CONN_13X2, P1 CONNECTOR_2, Q1 2N7002, U1 74XXX1G32, U2 74XXX1G32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

Commit message: Corrected note about bandwidth of amp circuit
Other:
- note added: "J1-J4 are C2000 Control Card Connectors"
Changed lines of the file:
@@
 Sheet 2 5
 Title "Connector, DAC, Power Input"
-Date "19 apr 2014"
+Date "20 oct 2015"
 Rev "1"
 Comp ""
@@
 	7150 4150 7050 4150
 Connection ~ 7050 4150
+Text Notes 3050 1700 0    60   ~ 0
+J1-J4 are C2000 Control Card Connectors
 $EndSCHEMATC
