File: Interface HW-04.sch (KiCad schematic (older format))
At the start: 0 parts

Commit message: Added buck converter to schematic, almost done
Parts:
- added C? (x7): CSMALL, ~, symbol CSMALL
- added L?: L_US, symbol L_US
- added R? (x4): R_US, ~, symbol R_US
- added U?: TPS5402, symbol TPS5402
Connections:
- net labels added: GND
- wire segments 0 -> 34

Commit message: Schematic before assigning ref des and netlisting
Parts:
- added D?: B130, symbol DIODE_SCHOTTKY
Connections:
- net labels added: +15V, 3V3
- wire segments 34 -> 36
Other:
- moved on the sheet: L?, R?, U?

Commit message: Started layout
Parts:
- gave numbers to parts that had none: 14
Changed lines of the file:
@@
 Sheet 5 5
 Title "Buck Conveter"
-Date "5 apr 2014"
+Date "9 apr 2014"
 Rev "1"
 Comp ""
@@
 $EndDescr
 $Comp
-L TPS5402 U?
+L TPS5402 U10
 U 1 1 5340586F
 P 5200 3600
-F 0 "U?" H 4950 4050 30  0000 L CNN
+F 0 "U10" H 4950 4050 30  0000 L CNN
 F 1 "TPS5402" H 4950 2600 30  0000 L CNN
 F 2 "" H 5200 3600 60  0000 C CNN
@@
 $EndComp
 $Comp
-L CSMALL C?
+L CSMALL C20
 U 1 1 5340587E
 P 5950 3450
-F 0 "C?" H 6000 3500 30  0000 L CNN
+F 0 "C20" H 6000 3500 30  0000 L CNN
 F 1 "CSMALL" H 6000 3450 30  0000 L CNN
 F 2 "~" H 5950 3450 60  0000 C CNN
@@
 $EndComp
 $Comp
-L R_US R?
+L R_US R22
 U 1 1 534058E6
 P 4050 4200
-F 0 "R?" H 4100 4250 30  0000 L CNN
+F 0 "R22" H 4100 4250 30  0000 L CNN
 F 1 "R_US" H 4100 4200 30  0000 L CNN
 F 2 "~" H 4050 4200 60  0000 C CNN
@@
 $EndComp
 $Comp
-L CSMALL C?
+L CSMALL C19
 U 1 1 5340594E
 P 4350 4300
-F 0 "C?" H 4400 4350 30  0000 L CNN
+F 0 "C19" H 4400 4350 30  0000 L CNN
 F 1 "CSMALL" H 4400 4300 30  0000 L CNN
 F 2 "~" H 4350 4300 60  0000 C CNN
@@
 Connection ~ 4350 4450
 $Comp
-L R_US R?
+L R_US R21
 U 1 1 53405966
 P 3700 3900
-F 0 "R?" H 3750 3950 30  0000 L CNN
+F 0 "R21" H 3750 3950 30  0000 L CNN
 F 1 "R_US" H 3750 3900 30  0000 L CNN
 F 2 "~" H 3700 3900 60  0000 C CNN
@@
 $EndComp
 $Comp
-L CSMALL C?
+L CSMALL C16
 U 1 1 5340596D
 P 3700 4300
-F 0 "C?" H 3750 4350 30  0000 L CNN
+F 0 "C16" H 3750 4350 30  0000 L CNN
 F 1 "CSMALL" H 3750 4300 30  0000 L CNN
 F 2 "~" H 3700 4300 60  0000 C CNN
@@
 	3700 4400 3700 4550
 $Comp
-L CSMALL C?
+L CSMALL C18
 U 1 1 534059A1
 P 4350 3250
-F 0 "C?" H 4400 3300 30  0000 L CNN
+F 0 "C18" H 4400 3300 30  0000 L CNN
 F 1 "CSMALL" H 4400 3250 30  0000 L CNN
 F 2 "~" H 4350 3250 60  0000 C CNN
@@
 	4600 3350 4650 3350
 $Comp
-L GND #PWR?
+L GND #PWR060
 U 1 1 534059B9
 P 3700 4550
-F 0 "#PWR?" H 3700 4550 30  0001 C CNN
+F 0 "#PWR060" H 3700 4550 30  0001 C CNN
 F 1 "GND" H 3700 4480 30  0001 C CNN
 F 2 "~" H 3700 4550 60  0000 C CNN
@@
 Connection ~ 3700 4450
 $Comp
-L GND #PWR?
+L GND #PWR061
 U 1 1 534059D8
 P 4050 3450
-F 0 "#PWR?" H 4050 3450 30  0001 C CNN
+F 0 "#PWR061" H 4050 3450 30  0001 C CNN
 F 1 "GND" H 4050 3380 30  0001 C CNN
 F 2 "~" H 4050 3450 60  0000 C CNN
@@
 	4050 3350 4050 3450
 $Comp
-L CSMALL C?
+L CSMALL C17
 U 1 1 534059F8
 P 4050 3250
-F 0 "C?" H 4100 3300 30  0000 L CNN
+F 0 "C17" H 4100 3300 30  0000 L CNN
 F 1 "CSMALL" H 4100 3250 30  0000 L CNN
 F 2 "~" H 4050 3250 60  0000 C CNN
@@
 	5950 3600 5950 3550
 $Comp
-L L_US L?
+L L_US L1
 U 1 1 53405A76
 P 6700 3600
-F 0 "L?" V 6900 3650 30  0000 L CNN
+F 0 "L1" V 6900 3650 30  0000 L CNN
 F 1 "L_US" V 6850 3600 30  0000 L CNN
 F 2 "" H 6700 3600 60  0000 C CNN
@@
 Connection ~ 5950 3600
 $Comp
-L CSMALL C?
+L CSMALL C21
 U 1 1 53405B03
 P 7650 3750
-F 0 "C?" H 7700 3800 30  0000 L CNN
+F 0 "C21" H 7700 3800 30  0000 L CNN
 F 1 "CSMALL" H 7700 3750 30  0000 L CNN
 F 2 "~" H 7650 3750 60  0000 C CNN
@@
 $EndComp
 $Comp
-L CSMALL C?
+L CSMALL C22
 U 1 1 53405B28
 P 7950 3750
-F 0 "C?" H 8000 3800 30  0000 L CNN
+F 0 "C22" H 8000 3800 30  0000 L CNN
 F 1 "CSMALL" H 8000 3750 30  0000 L CNN
 F 2 "~" H 7950 3750 60  0000 C CNN
@@
 $EndComp
 $Comp
-L GND #PWR?
+L GND #PWR062
 U 1 1 53405B4D
 P 7950 3950
-F 0 "#PWR?" H 7950 3950 30  0001 C CNN
+F 0 "#PWR062" H 7950 3950 30  0001 C CNN
 F 1 "GND" H 7950 3880 30  0001 C CNN
 F 2 "~" H 7950 3950 60  0000 C CNN
@@
 Connection ~ 7650 3600
 $Comp
-L R_US R?
+L R_US R23
 U 1 1 53405CF8
 P 7100 4200
-F 0 "R?" H 7150 4250 30  0000 L CNN
+F 0 "R23" H 7150 4250 30  0000 L CNN
 F 1 "R_US" H 7150 4200 30  0000 L CNN
 F 2 "~" H 7100 4200 60  0000 C CNN
@@
 $EndComp
 $Comp
-L R_US R?
+L R_US R24
 U 1 1 53405CFF
 P 7100 4700
-F 0 "R?" H 7150 4750 30  0000 L CNN
+F 0 "R24" H 7150 4750 30  0000 L CNN
 F 1 "R_US" H 7150 4700 30  0000 L CNN
 F 2 "~" H 7100 4700 60  0000 C CNN
@@
 $EndComp
 Wire Wire Line
-	7100 4100 7100 3600
-Connection ~ 7100 3600
-Wire Wire Line
 	6150 3900 6150 4450
 Wire Wire Line
 	6150 3900 5800 3900
 $Comp
-L GND #PWR?
+L GND #PWR063
 U 1 1 53405D7A
-P 7100 5050
-F 0 "#PWR?" H 7100 5050 30  0001 C CNN
-F 1 "GND" H 7100 4980 30  0001 C CNN
-F 2 "~" H 7100 5050 60  0000 C CNN
-F 3 "~" H 7100 5050 60  0000 C CNN
-	1    7100 5050
-	1    0    0    -1
-$EndComp
-Wire Wire Line
-	7100 5000 7100 5050
+P 7100 4950
+F 0 "#PWR063" H 7100 4950 30  0001 C CNN
+F 1 "GND" H 7100 4880 30  0001 C CNN
+F 2 "~" H 7100 4950 60  0000 C CNN
+F 3 "~" H 7100 4950 60  0000 C CNN
+	1    7100 4950
+	1    0    0    -1
+$EndComp
+Wire Wire Line
+	7100 4900 7100 4950
 Wire Wire Line
 	7100 4400 7100 4500
@@
 Connection ~ 7100 4450
 $Comp
-L DIODE_SCHOTTKY D?
+L DIODE_SCHOTTKY D1
 U 1 1 5340638A
 P 6350 3850
-F 0 "D?" V 6400 3950 30  0000 L CNN
+F 0 "D1" V 6400 3950 30  0000 L CNN
 F 1 "B130" V 6350 3950 30  0000 L CNN
 F 2 "" H 6350 3850 60  0000 C CNN
@@
 Connection ~ 6350 3600
 $Comp
-L GND #PWR?
+L GND #PWR064
 U 1 1 5340643D
 P 6350 4100
-F 0 "#PWR?" H 6350 4100 30  0001 C CNN
+F 0 "#PWR064" H 6350 4100 30  0001 C CNN
 F 1 "GND" H 6350 4030 30  0001 C CNN
 F 2 "~" H 6350 4100 60  0000 C CNN
@@
 	6350 4050 6350 4100
 $Comp
-L 3V3 #PWR?
+L 3V3 #PWR065
 U 1 1 53406BFD
 P 7950 3500
-F 0 "#PWR?" H 7950 3600 40  0001 C CNN
+F 0 "#PWR065" H 7950 3600 40  0001 C CNN
 F 1 "3V3" H 7950 3625 40  0000 C CNN
 F 2 "~" H 7950 3500 60  0000 C CNN
@@
 Connection ~ 7950 3600
 $Comp
-L +15V #PWR?
+L +15V #PWR066
 U 1 1 53406C3C
 P 4050 3000
-F 0 "#PWR?" H 4050 2950 20  0001 C CNN
+F 0 "#PWR066" H 4050 2950 20  0001 C CNN
 F 1 "+15V" H 4050 3100 30  0000 C CNN
 F 2 "~" H 4050 3000 60  0000 C CNN
@@
 $EndComp
 Connection ~ 4050 3100
+Wire Wire Line
+	7100 4000 7100 3600
+Connection ~ 7100 3600
 $EndSCHEMATC

Commit message: Added a cap to ref, chages buck converter caps, more routing, didn't pull in netlist
Parts:
- C17, C21, C22: value CSMALL -> 10uF
Changed lines of the file:
@@
 Sheet 5 5
 Title "Buck Conveter"
-Date "9 apr 2014"
+Date "16 apr 2014"
 Rev "1"
 Comp ""
@@
 	4600 3350 4650 3350
 $Comp
-L GND #PWR060
+L GND #PWR061
 U 1 1 534059B9
 P 3700 4550
-F 0 "#PWR060" H 3700 4550 30  0001 C CNN
+F 0 "#PWR061" H 3700 4550 30  0001 C CNN
 F 1 "GND" H 3700 4480 30  0001 C CNN
 F 2 "~" H 3700 4550 60  0000 C CNN
@@
 Connection ~ 3700 4450
 $Comp
-L GND #PWR061
+L GND #PWR062
 U 1 1 534059D8
 P 4050 3450
-F 0 "#PWR061" H 4050 3450 30  0001 C CNN
+F 0 "#PWR062" H 4050 3450 30  0001 C CNN
 F 1 "GND" H 4050 3380 30  0001 C CNN
 F 2 "~" H 4050 3450 60  0000 C CNN
@@
 P 4050 3250
 F 0 "C17" H 4100 3300 30  0000 L CNN
-F 1 "CSMALL" H 4100 3250 30  0000 L CNN
+F 1 "10uF" H 4100 3250 30  0000 L CNN
 F 2 "~" H 4050 3250 60  0000 C CNN
 F 3 "~" H 4050 3250 60  0000 C CNN
@@
 P 7650 3750
 F 0 "C21" H 7700 3800 30  0000 L CNN
-F 1 "CSMALL" H 7700 3750 30  0000 L CNN
+F 1 "10uF" H 7700 3750 30  0000 L CNN
 F 2 "~" H 7650 3750 60  0000 C CNN
 F 3 "~" H 7650 3750 60  0000 C CNN
@@
 P 7950 3750
 F 0 "C22" H 8000 3800 30  0000 L CNN
-F 1 "CSMALL" H 8000 3750 30  0000 L CNN
+F 1 "10uF" H 8000 3750 30  0000 L CNN
 F 2 "~" H 7950 3750 60  0000 C CNN
 F 3 "~" H 7950 3750 60  0000 C CNN
@@
 $EndComp
 $Comp
-L GND #PWR062
+L GND #PWR063
 U 1 1 53405B4D
 P 7950 3950
-F 0 "#PWR062" H 7950 3950 30  0001 C CNN
+F 0 "#PWR063" H 7950 3950 30  0001 C CNN
 F 1 "GND" H 7950 3880 30  0001 C CNN
 F 2 "~" H 7950 3950 60  0000 C CNN
@@
 	6150 3900 5800 3900
 $Comp
-L GND #PWR063
+L GND #PWR064
 U 1 1 53405D7A
 P 7100 4950
-F 0 "#PWR063" H 7100 4950 30  0001 C CNN
+F 0 "#PWR064" H 7100 4950 30  0001 C CNN
 F 1 "GND" H 7100 4880 30  0001 C CNN
 F 2 "~" H 7100 4950 60  0000 C CNN
@@
 Connection ~ 6350 3600
 $Comp
-L GND #PWR064
+L GND #PWR065
 U 1 1 5340643D
 P 6350 4100
-F 0 "#PWR064" H 6350 4100 30  0001 C CNN
+F 0 "#PWR065" H 6350 4100 30  0001 C CNN
 F 1 "GND" H 6350 4030 30  0001 C CNN
 F 2 "~" H 6350 4100 60  0000 C CNN
@@
 	6350 4050 6350 4100
 $Comp
-L 3V3 #PWR065
+L 3V3 #PWR066
 U 1 1 53406BFD
 P 7950 3500
-F 0 "#PWR065" H 7950 3600 40  0001 C CNN
+F 0 "#PWR066" H 7950 3600 40  0001 C CNN
 F 1 "3V3" H 7950 3625 40  0000 C CNN
 F 2 "~" H 7950 3500 60  0000 C CNN
@@
 Connection ~ 7950 3600
 $Comp
-L +15V #PWR066
+L +15V #PWR067
 U 1 1 53406C3C
 P 4050 3000
-F 0 "#PWR066" H 4050 2950 20  0001 C CNN
+F 0 "#PWR067" H 4050 2950 20  0001 C CNN
 F 1 "+15V" H 4050 3100 30  0000 C CNN
 F 2 "~" H 4050 3000 60  0000 C CNN
