File: Interface HW.kicad_pcb (KiCad board)
At the start: 2 copper layers, 50 x 50 mm, 90 parts, among them J1 CONN_8, J2 CONN_8, J3 CONN_8, J4 CONN_8, J5 TE: 640456-3, J6 CONN_13X2, J7 TERM_3, J8 TERM-3, P1 CONNECTOR_2, Q1 2N7002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

Commit message: Updated schematic
Parts:
- moved L1 2.77 mm to (115.2, 125.0)
Routing:
- net N-0000068: track 16.7 -> 18.5 mm
- net /Interface HW-01/GPIO_12: track 85.7 -> 86.3 mm
- net GND: vias 17 -> 18
- net (no net): vias 0 -> 1
- added copper zone on F.Cu, net 3V3
- added copper zone on B.Cu, net GND
- added copper zone on F.Cu, net GND
- added copper zone on F.Cu, net N-0000068

Commit message: Created gerber files for release
Routing:
- net /Interface HW-01/SPICLK_A: track 39.6 -> 39.0 mm
Changed lines of the file:
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@@
     (thickness 1.6)
     (drawings 5)
-    (tracks 721)
+    (tracks 722)
     (zones 0)
     (modules 90)
@@
   (layers
     (15 F.Cu signal)
-    (0 B.Cu signal hide)
+    (0 B.Cu signal)
     (16 B.Adhes user hide)
     (17 F.Adhes user hide)
@@
   (segment (start 119.1 117.3) (end 119.1 113.25) (width 0.1524) (layer F.Cu) (net 5))
   (segment (start 119.35 117.55) (end 119.1 117.3) (width 0.1524) (layer F.Cu) (net 5))
-  (segment (start 118.75 115.05) (end 114 115.05) (width 0.1524) (layer B.Cu) (net 6))
-  (segment (start 118.75 115.05) (end 119.6 114.2) (width 0.1524) (layer B.Cu) (net 6))
-  (segment (start 119.6 114.2) (end 119.6 110.75) (width 0.1524) (layer B.Cu) (net 6))
-  (segment (start 119.6 110.75) (end 120.1 110.25) (width 0.1524) (layer B.Cu) (net 6))
+  (segment (start 106.22 115.05) (end 106.77 114.5) (width 0.1524) (layer F.Cu) (net 6))
+  (segment (start 118.35 114.5) (end 114 114.5) (width 0.1524) (layer B.Cu) (net 6))
+  (via (at 114 114.5) (size 0.889) (layers F.Cu B.Cu) (net 6))
+  (segment (start 127.34 110.25) (end 128.54 111.45) (width 0.1524) (layer B.Cu) (net 6) (status 10))
   (segment (start 120.1 110.25) (end 127.34 110.25) (width 0.1524) (layer B.Cu) (net 6))
-  (segment (start 128.54 111.45) (end 127.34 110.25) (width 0.1524) (layer B.Cu) (net 6) (status 10))
-  (segment (start 114 115.05) (end 106.22 115.05) (width 0.1524) (layer F.Cu) (net 6) (status 20))
-  (via (at 114 115.05) (size 0.889) (layers F.Cu B.Cu) (net 6))
+  (segment (start 119.6 110.75) (end 120.1 110.25) (width 0.1524) (layer B.Cu) (net 6))
+  (segment (start 119.6 113.25) (end 119.6 110.75) (width 0.1524) (layer B.Cu) (net 6))
+  (segment (start 119.6 113.25) (end 118.35 114.5) (width 0.1524) (layer B.Cu) (net 6))
+  (segment (start 106.77 114.5) (end 114 114.5) (width 0.1524) (layer F.Cu) (net 6))
   (segment (start 128.54 111.45) (end 128.54 111.91) (width 0.1524) (layer F.Cu) (net 6) (status 30))
   (segment (start 125.45 117.25) (end 125.35 117.35) (width 0.1524) (layer F.Cu) (net 6))
@@
   (segment (start 123.6 122.2104) (end 121.15 122.2104) (width 0.1524) (layer F.Cu) (net 7))
   (segment (start 109.48 120.13) (end 106.22 120.13) (width 0.1524) (layer F.Cu) (net 7) (status 20))
-  (segment (start 115.03 116.6475) (end 115.03 115.77) (width 0.1524) (layer F.Cu) (net 8) (status 10))
-  (segment (start 120.95 113.65) (end 121.55 114.25) (width 0.1524) (layer F.Cu) (net 8))
-  (segment (start 120.9 113.65) (end 120.95 113.65) (width 0.1524) (layer F.Cu) (net 8))
+  (segment (start 115 115.35) (end 119.2 115.35) (width 0.1524) (layer B.Cu) (net 8))
+  (segment (start 114.98 115.37) (end 115 115.35) (width 0.1524) (layer F.Cu) (net 8))
+  (via (at 115 115.35) (size 0.889) (layers F.Cu B.Cu) (net 8))
   (via (at 120.9 113.65) (size 0.889) (layers F.Cu B.Cu) (net 8))
-  (segment (start 118.8 115.75) (end 120.9 113.65) (width 0.1524) (layer B.Cu) (net 8))
-  (segment (start 115.05 115.75) (end 118.8 115.75) (width 0.1524) (layer B.Cu) (net 8))
-  (via (at 115.05 115.75) (size 0.889) (layers F.Cu B.Cu) (net 8))
-  (segment (start 115.03 115.77) (end 115.05 115.75) (width 0.1524) (layer F.Cu) (net 8))
+  (segment (start 120.9 113.65) (end 120.95 113.65) (width 0.1524) (layer F.Cu) (net 8))
+  (segment (start 121.55 114.25) (end 120.95 113.65) (width 0.1524) (layer F.Cu) (net 8))
+  (segment (start 114.98 115.37) (end 115.03 116.6475) (width 0.1524) (layer F.Cu) (net 8) (status 10))
+  (segment (start 119.2 115.35) (end 120.9 113.65) (width 0.1524) (layer B.Cu) (net 8))
   (segment (start 103.68 117.59) (end 104.97 116.3) (width 0.1524) (layer B.Cu) (net 8) (status 10))
-  (segment (start 111.6975 116.6475) (end 115.03 116.6475) (width 0.1524) (layer F.Cu) (net 8) (status 20))
-  (segment (start 111.35 116.3) (end 111.6975 116.6475) (width 0.1524) (layer F.Cu) (net 8))
-  (segment (start 109 116.3) (end 111.35 116.3) (width 0.1524) (layer F.Cu) (net 8))
-  (via (at 109 116.3) (size 0.889) (layers F.Cu B.Cu) (net 8))
   (segment (start 104.97 116.3) (end 109 116.3) (width 0.1524) (layer B.Cu) (net 8))
+  (via (at 109 116.3) (size 0.889) (layers F.Cu B.Cu) (net 8))
+  (segment (start 109 116.3) (end 111.35 116.3) (width 0.1524) (layer F.Cu) (net 8))
+  (segment (start 111.35 116.3) (end 111.6975 116.6475) (width 0.1524) (layer F.Cu) (net 8))
+  (segment (start 111.6975 116.6475) (end 115.03 116.6475) (width 0.1524) (layer F.Cu) (net 8) (status 20))
   (segment (start 126 111.45) (end 126 113.1) (width 0.1524) (layer F.Cu) (net 8) (status 10))
   (segment (start 126 113.1) (end 124.85 114.25) (width 0.1524) (layer F.Cu) (net 8))
